Commit message: Add files via upload

File: robot_core.xacro (robot description, xacro)
@@ -194,46 +194,79 @@
     </xacro:inertial_box>
 </link>
-<!-- ARM -->
-<!-- <joint name="arm_joint" type="revolute">
-    <parent link="arm_base"/>
-    <child link="arm_link"/>
-    <origin xyz="0 0 0.05" rpy="0 0 0"/>
-    <axis xyz="0 1 0"/> <limit lower="-1.57" upper="1.57" effort="10" velocity="1.0"/>
-</joint>
-<link name="arm_link">
-    <visual>
-        <origin xyz="0.1 0 0" rpy="0 0 0"/>
-        <geometry>
-            <box size="0.2 0.04 0.04"/>
-        </geometry>
-        <material name="white"/>
-    </visual>
-</link> -->
-<!-- CASTER WHEEL -->
-<!-- <joint name="caster_wheel_joint" type="fixed">
-    <parent link="chassis"/>
-    <child link="caster_wheel"/>
-    <origin xyz="0.24 0 0" rpy="0 0 0"/>
-</joint>
-<link name="caster_wheel">
-    <visual>
-        <geometry>
-            <sphere radius="0.05" />
-        </geometry>
-        <material name="black"/>
-    </visual>
-    <collision>
-        <geometry>
-            <sphere radius="0.05" />
-        </geometry>
-    </collision>
-    <xacro:inertial_sphere mass="0.1" radius="0.05">
-            <origin xyz="0 0 0" rpy="0 0 0"/>
-    </xacro:inertial_sphere>
-</link>
-<gazebo reference="caster_wheel">
-    <material>Gazebo/Black</material>
-    <mu1 value="0.001"/>
-    <mu2 value="0.001"/>
-</gazebo> -->
+<!-- ARM L-->
+<joint name="arm_slide_joint_L" type="prismatic">
+    <parent link="arm_base2"/>
+    <child link="arm_dummy_link"/>
+    <origin xyz="0 -0.2475 0" rpy="0 0 0"/>
+    <axis xyz="0 1 0"/>
+    <limit lower="0" upper="0.235" effort="100" velocity="1.0"/>
+</joint>
+<link name="arm_dummy_link">
+    <xacro:inertial_box mass="0.01" x="0.01" y="0.01" z="0.01">
+        <origin xyz="0 0 0" rpy="0 0 0"/>
+    </xacro:inertial_box>
+</link>
+<joint name="arm_rotate_joint_L" type="revolute">
+    <parent link="arm_dummy_link"/>
+    <child link="arm_link_L"/>
+    <origin xyz="0 0 0" rpy="0 0 0"/>
+    <axis xyz="0 0 1"/>
+    <limit lower="-0.785" upper="0.785" effort="100" velocity="1.0"/>
+</joint>
+<link name="arm_link_L">
+    <visual>
+        <origin xyz="0.075 0 0" rpy="0 0 0"/>
+        <geometry>
+            <box size="0.15 0.025 0.05"/>
+        </geometry>
+        <material name="white"/>
+    </visual>
+    <collision>
+        <origin xyz="0.075 0 0" rpy="0 0 0"/>
+        <geometry>
+            <box size="0.15 0.025 0.05"/>
+        </geometry>
+    </collision>
+    <xacro:inertial_box mass="0.5" x="0.15" y="0.025" z="0.05">
+        <origin xyz="0 0 0" rpy="0 0 0"/>
+    </xacro:inertial_box>
+</link>
+<!-- ARM R -->
+<joint name="arm_slide_joint_R" type="prismatic">
+    <parent link="arm_base2"/>
+    <child link="arm_dummy_link_R"/>
+    <origin xyz="0 0.2475 0" rpy="0 0 0"/>
+    <axis xyz="0 1 0"/>
+    <limit lower="-0.235" upper="0" effort="100" velocity="1.0"/>
+</joint>
+<link name="arm_dummy_link_R">
+    <xacro:inertial_box mass="0.01" x="0.01" y="0.01" z="0.01">
+        <origin xyz="0 0 0" rpy="0 0 0"/>
+    </xacro:inertial_box>
+</link>
+<joint name="arm_rotate_joint_R" type="revolute">
+    <parent link="arm_dummy_link_R"/>
+    <child link="arm_link_R"/>
+    <origin xyz="0 0 0" rpy="0 0 0"/>
+    <axis xyz="0 0 1"/>
+    <limit lower="-0.785" upper="0.785" effort="100" velocity="1.0"/>
+</joint>
+<link name="arm_link_R">
+    <visual>
+        <origin xyz="0.075 0 0" rpy="0 0 0"/>
+        <geometry>
+            <box size="0.15 0.025 0.05"/>
+        </geometry>
+        <material name="white"/>
+    </visual>
+    <collision>
+        <origin xyz="0.075 0 0" rpy="0 0 0"/>
+        <geometry>
+            <box size="0.15 0.025 0.05"/>
+        </geometry>
+    </collision>
+    <xacro:inertial_box mass="0.5" x="0.15" y="0.025" z="0.05">
+        <origin xyz="0.075 0 0" rpy="0 0 0"/>
+    </xacro:inertial_box>
+</link>
 </robot>
