Commit message: Add files via upload

File: description/gazebo_control.xacro (robot description, xacro)
@@ -3,13 +3,13 @@
   <gazebo>
       <plugin name='diff_drive' filename='libgazebo_ros_diff_drive.so'>
-          <!-- Wheel Information -->
+          <num_wheel_pairs>2</num_wheel_pairs>
+          <left_joint>front_left_wheel_joint</left_joint>
+          <right_joint>front_right_wheel_joint</right_joint>
           <left_joint>back_left_wheel_joint</left_joint>
           <right_joint>back_right_wheel_joint</right_joint>
-          <wheel_separation>0.35</wheel_separation>
+          <wheel_separation>0.34</wheel_separation>
           <wheel_diameter>0.1</wheel_diameter>
-          <!-- Limits -->
           <max_wheel_torque>200</max_wheel_torque>
           <max_wheel_acceleration>10.0</max_wheel_acceleration>
-          <!-- Output -->
           <odometry_frame>odom</odometry_frame>
           <robot_base_frame>base_link</robot_base_frame>

File: description/robot_core.xacro (robot description, xacro)
@@ -91,5 +91,5 @@
     <child link="front_right_wheel"/>
     <origin xyz="0.075 -0.17 0.05" rpy="${pi/2} 0 0"/>
-    <axis xyz="0 0 1"/>
+    <axis xyz="0 0 -1"/>
 </joint>
 <link name="front_right_wheel">
@@ -113,5 +113,5 @@
     <child link="back_right_wheel"/>
     <origin xyz="-0.075 -0.17 0.05" rpy="${pi/2} 0 0"/>
-    <axis xyz="0 0 1"/>
+    <axis xyz="0 0 -1"/>
 </joint>
 <link name="back_right_wheel">
@@ -205,4 +205,11 @@
     </xacro:inertial_box>
 </link>
+ <gazebo reference="arm_link_L">
+        <mu1>100.0</mu1>
+        <mu2>100.0</mu2>
+        <kp>1000000.0</kp>
+        <kd>1.0</kd>
+        <material>Gazebo/White</material>
+</gazebo>
 <joint name="arm_slide_joint_R" type="prismatic">
     <parent link="arm_base2"/>
@@ -230,3 +237,10 @@
     </xacro:inertial_box>
 </link>
+<gazebo reference="arm_link_R">
+        <mu1>100.0</mu1>
+        <mu2>100.0</mu2>
+        <kp>1000000.0</kp>
+        <kd>1.0</kd>
+        <material>Gazebo/White</material>
+</gazebo>
 </robot>

Commit message: Add files via upload

File: description/gazebo_control.xacro (robot description, xacro)
@@ -10,5 +10,5 @@
           <wheel_separation>0.34</wheel_separation>
           <wheel_diameter>0.1</wheel_diameter>
-          <max_wheel_torque>200</max_wheel_torque>
+          <max_wheel_torque>400</max_wheel_torque>
           <max_wheel_acceleration>10.0</max_wheel_acceleration>
           <odometry_frame>odom</odometry_frame>

File: description/robot_core.xacro (robot description, xacro)
@@ -36,5 +36,5 @@
         </geometry>
     </collision>
-    <xacro:inertial_box mass="3" x="0.3" y="0.3" z="0.15">
+    <xacro:inertial_box mass="20" x="0.3" y="0.3" z="0.15">
         <origin xyz="0 0 0.075" rpy="0 0 0"/>
     </xacro:inertial_box>
@@ -185,5 +185,5 @@
     <origin xyz="0 -0.25375 0" rpy="0 0 0"/>
     <axis xyz="0 1 0"/>
-    <limit lower="0" upper="0.25375" effort="100" velocity="1.0"/>
+    <limit lower="0" upper="0.25375" effort="200" velocity="1.0"/>
 </joint>
 <link name="arm_link_L">
@@ -212,4 +212,5 @@
         <material>Gazebo/White</material>
 </gazebo>
+<!-- ARM R -->
 <joint name="arm_slide_joint_R" type="prismatic">
     <parent link="arm_base2"/>
@@ -217,5 +218,5 @@
     <origin xyz="0 0.25375 0" rpy="0 0 0"/>
     <axis xyz="0 1 0"/>
-    <limit lower="-0.25375" upper="0" effort="100" velocity="1.0"/>
+    <limit lower="-0.25375" upper="0" effort="200" velocity="1.0"/>
 </joint>
 <link name="arm_link_R">

Commit message: Add files via upload

File: description/gazebo_control.xacro (robot description, xacro)
@@ -11,5 +11,5 @@
           <wheel_diameter>0.1</wheel_diameter>
           <max_wheel_torque>400</max_wheel_torque>
-          <max_wheel_acceleration>10.0</max_wheel_acceleration>
+          <max_wheel_acceleration>50.0</max_wheel_acceleration>
           <odometry_frame>odom</odometry_frame>
           <robot_base_frame>base_link</robot_base_frame>

File: description/robot_core.xacro (robot description, xacro)
@@ -131,4 +131,20 @@
     </xacro:inertial_cylinder>
 </link>
+<gazebo reference="front_left_wheel">
+    <mu1>0.2</mu1>
+    <mu2>0.2</mu2>
+</gazebo>
+<gazebo reference="back_left_wheel">
+    <mu1>0.2</mu1>
+    <mu2>0.2</mu2>
+</gazebo>
+<gazebo reference="front_right_wheel">
+    <mu1>0.2</mu1>
+    <mu2>0.2</mu2>
+</gazebo>
+<gazebo reference="back_right_wheel">
+    <mu1>0.2</mu1>
+    <mu2>0.2</mu2>
+</gazebo>
 <joint name="arm_base1_joint" type="fixed">
     <parent link="chassis"/>
@@ -159,5 +175,5 @@
     <origin xyz="0.05 0 0.025" rpy="0 0 0"/>
     <axis xyz="0 0 1"/>
-    <limit lower="0" upper="0.2" effort="100" velocity="1.0"/>
+    <limit lower="0" upper="0.2" effort="500" velocity="1.0"/>
 </joint>
 <link name="arm_base2">
@@ -165,15 +181,15 @@
         <origin xyz="0 0 0" rpy="0 0 0"/>
         <geometry>
-            <box size="0.05 0.52 0.05"/>
-        </geometry>
-        <material name="white"/>
-    </visual>
-    <collision>
-        <origin xyz="0 0 0" rpy="0 0 0"/>
-        <geometry>
-            <box size="0.05 0.52 0.05"/>
-        </geometry>
-    </collision>
-    <xacro:inertial_box mass="0.2" x="0.05" y="0.52" z="0.05">
+            <box size="0.05 0.54 0.05"/>
+        </geometry>
+        <material name="white"/>
+    </visual>
+    <collision>
+        <origin xyz="0 0 0" rpy="0 0 0"/>
+        <geometry>
+            <box size="0.05 0.54 0.05"/>
+        </geometry>
+    </collision>
+    <xacro:inertial_box mass="0.2" x="0.05" y="0.54" z="0.05">
         <origin xyz="0 0 0" rpy="0 0 0"/>
     </xacro:inertial_box>
@@ -183,7 +199,7 @@
     <parent link="arm_base2"/>
     <child link="arm_link_L"/>
-    <origin xyz="0 -0.25375 0" rpy="0 0 0"/>
+    <origin xyz="0 -0.26375 0" rpy="0 0 0"/>
     <axis xyz="0 1 0"/>
-    <limit lower="0" upper="0.25375" effort="200" velocity="1.0"/>
+    <limit lower="0" upper="0.26375" effort="400" velocity="1.0"/>
 </joint>
 <link name="arm_link_L">
@@ -216,7 +232,7 @@
     <parent link="arm_base2"/>
     <child link="arm_link_R"/>
-    <origin xyz="0 0.25375 0" rpy="0 0 0"/>
+    <origin xyz="0 0.26375 0" rpy="0 0 0"/>
     <axis xyz="0 1 0"/>
-    <limit lower="-0.25375" upper="0" effort="200" velocity="1.0"/>
+    <limit lower="-0.26375" upper="0" effort="400" velocity="1.0"/>
 </joint>
 <link name="arm_link_R">

Commit message: Add files via upload

File: description/gazebo_control.xacro (robot description, xacro)
@@ -10,6 +10,6 @@
           <wheel_separation>0.34</wheel_separation>
           <wheel_diameter>0.1</wheel_diameter>
-          <max_wheel_torque>400</max_wheel_torque>
-          <max_wheel_acceleration>50.0</max_wheel_acceleration>
+          <max_wheel_torque>1000</max_wheel_torque>
+          <max_wheel_acceleration>10</max_wheel_acceleration>
           <odometry_frame>odom</odometry_frame>
           <robot_base_frame>base_link</robot_base_frame>

File: description/robot_core.xacro (robot description, xacro)
@@ -43,4 +43,5 @@
     <material>Gazebo/White</material>
 </gazebo>
+<!-- front_left_wheel_joint -->
 <joint name="front_left_wheel_joint" type="continuous">
     <parent link="base_link"/>
@@ -61,8 +62,9 @@
         </geometry>
     </collision>
-    <xacro:inertial_cylinder mass="0.1" length="0.04" radius="0.05">
-        <origin xyz="0 0 0" rpy="0 0 0"/>
-    </xacro:inertial_cylinder>
-</link>
+    <xacro:inertial_cylinder mass="1" length="0.04" radius="0.05">
+        <origin xyz="0 0 0" rpy="0 0 0"/>
+    </xacro:inertial_cylinder>
+</link>
+<!-- back_left_wheel_joint -->
 <joint name="back_left_wheel_joint" type="continuous">
     <parent link="base_link"/>
@@ -83,8 +85,9 @@
         </geometry>
     </collision>
-    <xacro:inertial_cylinder mass="0.1" length="0.04" radius="0.05">
-        <origin xyz="0 0 0" rpy="0 0 0"/>
-    </xacro:inertial_cylinder>
-</link>
+    <xacro:inertial_cylinder mass="1" length="0.04" radius="0.05">
+        <origin xyz="0 0 0" rpy="0 0 0"/>
+    </xacro:inertial_cylinder>
+</link>
+<!-- front_right_wheel_joint -->
 <joint name="front_right_wheel_joint" type="continuous">
     <parent link="base_link"/>
@@ -105,8 +108,9 @@
         </geometry>
     </collision>
-    <xacro:inertial_cylinder mass="0.1" length="0.04" radius="0.05">
-        <origin xyz="0 0 0" rpy="0 0 0"/>
-    </xacro:inertial_cylinder>
-</link>
+    <xacro:inertial_cylinder mass="1" length="0.04" radius="0.05">
+        <origin xyz="0 0 0" rpy="0 0 0"/>
+    </xacro:inertial_cylinder>
+</link>
+<!-- back_right_wheel_joint -->
 <joint name="back_right_wheel_joint" type="continuous">
     <parent link="base_link"/>
@@ -127,22 +131,22 @@
         </geometry>
     </collision>
-    <xacro:inertial_cylinder mass="0.1" length="0.04" radius="0.05">
+    <xacro:inertial_cylinder mass="1" length="0.04" radius="0.05">
         <origin xyz="0 0 0" rpy="0 0 0"/>
     </xacro:inertial_cylinder>
 </link>
 <gazebo reference="front_left_wheel">
-    <mu1>0.2</mu1>
+    <mu1>2</mu1>
     <mu2>0.2</mu2>
 </gazebo>
 <gazebo reference="back_left_wheel">
-    <mu1>0.2</mu1>
+    <mu1>2</mu1>
     <mu2>0.2</mu2>
 </gazebo>
 <gazebo reference="front_right_wheel">
-    <mu1>0.2</mu1>
+    <mu1>2</mu1>
     <mu2>0.2</mu2>
 </gazebo>
 <gazebo reference="back_right_wheel">
-    <mu1>0.2</mu1>
+    <mu1>2</mu1>
     <mu2>0.2</mu2>
 </gazebo>
