Commit message: Add files via upload

File: description/robot_core.xacro (robot description, xacro)
@@ -157,7 +157,7 @@
     <parent link="arm_base1"/>
     <child link="arm_base2"/>
-    <origin xyz="0.05 0 0.15" rpy="0 0 0"/>
+    <origin xyz="0.05 0 0.025" rpy="0 0 0"/>
     <axis xyz="0 0 1"/>
-    <limit lower="-0.1" upper="0.1" effort="100" velocity="1.0"/>
+    <limit lower="0" upper="0.2" effort="100" velocity="1.0"/>
 </joint>
 <link name="arm_base2">
@@ -183,7 +183,7 @@
     <parent link="arm_base2"/>
     <child link="arm_link_L"/>
-    <origin xyz="0 -0.2475 0" rpy="0 0 0"/>
+    <origin xyz="0 -0.25375 0" rpy="0 0 0"/>
     <axis xyz="0 1 0"/>
-    <limit lower="0" upper="0.235" effort="100" velocity="1.0"/>
+    <limit lower="0" upper="0.25375" effort="100" velocity="1.0"/>
 </joint>
 <link name="arm_link_L">
@@ -191,15 +191,15 @@
         <origin xyz="0.075 0 0" rpy="0 0 0"/>
         <geometry>
-            <box size="0.15 0.025 0.05"/>
-        </geometry>
-        <material name="white"/>
-    </visual>
-    <collision>
-        <origin xyz="0.075 0 0" rpy="0 0 0"/>
-        <geometry>
-            <box size="0.15 0.025 0.05"/>
-        </geometry>
-    </collision>
-    <xacro:inertial_box mass="0.1" x="0.15" y="0.025" z="0.05">
+            <box size="0.15 0.0125 0.05"/>
+        </geometry>
+        <material name="white"/>
+    </visual>
+    <collision>
+        <origin xyz="0.075 0 0" rpy="0 0 0"/>
+        <geometry>
+            <box size="0.15 0.0125 0.05"/>
+        </geometry>
+    </collision>
+    <xacro:inertial_box mass="0.1" x="0.15" y="0.0125" z="0.05">
         <origin xyz="0.075 0 0" rpy="0 0 0"/>
     </xacro:inertial_box>
@@ -215,7 +215,7 @@
     <parent link="arm_base2"/>
     <child link="arm_link_R"/>
-    <origin xyz="0 0.2475 0" rpy="0 0 0"/>
+    <origin xyz="0 0.25375 0" rpy="0 0 0"/>
     <axis xyz="0 1 0"/>
-    <limit lower="-0.235" upper="0" effort="100" velocity="1.0"/>
+    <limit lower="-0.25375" upper="0" effort="100" velocity="1.0"/>
 </joint>
 <link name="arm_link_R">
@@ -223,15 +223,15 @@
         <origin xyz="0.075 0 0" rpy="0 0 0"/>
         <geometry>
-            <box size="0.15 0.025 0.05"/>
-        </geometry>
-        <material name="white"/>
-    </visual>
-    <collision>
-        <origin xyz="0.075 0 0" rpy="0 0 0"/>
-        <geometry>
-            <box size="0.15 0.025 0.05"/>
-        </geometry>
-    </collision>
-    <xacro:inertial_box mass="0.1" x="0.15" y="0.025" z="0.05">
+            <box size="0.15 0.0125 0.05"/>
+        </geometry>
+        <material name="white"/>
+    </visual>
+    <collision>
+        <origin xyz="0.075 0 0" rpy="0 0 0"/>
+        <geometry>
+            <box size="0.15 0.0125 0.05"/>
+        </geometry>
+    </collision>
+    <xacro:inertial_box mass="0.1" x="0.15" y="0.0125" z="0.05">
         <origin xyz="0.075 0 0" rpy="0 0 0"/>
     </xacro:inertial_box>

Commit message: Add files via upload

File: description/robot_core.xacro (robot description, xacro)
@@ -180,5 +180,5 @@
     <origin xyz="0.05 0 0.025" rpy="0 0 0"/>
     <axis xyz="0 0 1"/>
-    <limit lower="0" upper="0.2" effort="500" velocity="1.0"/>
+    <limit lower="0" upper="0.2" effort="1000" velocity="1.0"/>
 </joint>
 <link name="arm_base2">
@@ -206,5 +206,5 @@
     <origin xyz="0 -0.26375 0" rpy="0 0 0"/>
     <axis xyz="0 1 0"/>
-    <limit lower="0" upper="0.26375" effort="400" velocity="1.0"/>
+    <limit lower="0" upper="0.26375" effort="1000" velocity="1.0"/>
 </joint>
 <link name="arm_link_L">
@@ -239,5 +239,5 @@
     <origin xyz="0 0.26375 0" rpy="0 0 0"/>
     <axis xyz="0 1 0"/>
-    <limit lower="-0.26375" upper="0" effort="400" velocity="1.0"/>
+    <limit lower="-0.26375" upper="0" effort="1000" velocity="1.0"/>
 </joint>
 <link name="arm_link_R">
